Commit message: Edicion del xacro para adaptar a Gazebo

File: KUKA_10/kr10_description/urdf/kr10_macro.xacro (robot description, xacro)
@@ -17,4 +17,9 @@
         </geometry>
       </collision>
+      <inertial>
+        <mass value="23.085357"/>
+        <origin rpy="0.0 0.0 0.0" xyz="0.007579 0.000017 0.180670"/>
+        <inertia ixx="0.343576" ixy="-0.000062" ixz="-0.002079" iyy="0.336217" iyz="-0.000014" izz="0.334050"/>
+      </inertial>
     </link>
     <link name="${prefix}link_1">
@@ -32,4 +37,9 @@
         </geometry>
       </collision>
+      <inertial>
+        <mass value="45.357763"/>
+        <origin rpy="0.0 0.0 0.0" xyz="0.085479 -0.002547 -0.040488"/>
+        <inertia ixx="0.839141" ixy="0.022637" ixz="0.162457" iyy="1.030146" iyz="0.027416" izz="1.064698"/>
+      </inertial>
     </link>
     <link name="${prefix}link_2">
@@ -47,4 +57,9 @@
         </geometry>
       </collision>
+      <inertial>
+        <mass value="51.266495"/>
+        <origin rpy="0.0 0.0 0.0" xyz="-0.000002 0.264164 0.347704"/>
+        <inertia ixx="5.272800" ixy="0.000010" ixz="0.000017" iyy="5.536809" iyz="-0.008261" izz="0.486191"/>
+      </inertial>
     </link>
     <link name="${prefix}link_3">
@@ -62,4 +77,9 @@
         </geometry>
       </collision>
+      <inertial>
+        <mass value="19.754401"/>
+        <origin rpy="0.0 0.0 0.0" xyz="-0.000255 0.016478 -0.003819"/>
+        <inertia ixx="0.249388" ixy="-0.004901" ixz="0.004825" iyy="0.211780" iyz="0.000574" izz="0.238488"/>
+      </inertial>
     </link>
     <link name="${prefix}link_4">
@@ -77,4 +97,9 @@
         </geometry>
       </collision>
+      <inertial>
+        <mass value="15.287896"/>
+        <origin rpy="0.0 0.0 0.0" xyz="-0.015515 0.000164 0.340348"/>
+        <inertia ixx="0.331593" ixy="0.000055" ixz="-0.010688" iyy="0.320895" iyz="0.000058" izz="0.086557"/>
+      </inertial>
     </link>
     <link name="${prefix}link_5">
@@ -92,4 +117,9 @@
         </geometry>
       </collision>
+      <inertial>
+        <mass value="0.548088"/>
+        <origin rpy="0.0 0.0 0.0" xyz="0.000000 -0.000347 0.023671"/>
+        <inertia ixx="0.000876" ixy="0.000000" ixz="0.000000" iyy="0.000889" iyz="0.000005" izz="0.000412"/>
+      </inertial>
     </link>
     <link name="${prefix}link_6">
@@ -107,4 +137,9 @@
         </geometry>
       </collision>
+      <inertial>
+        <mass value="0.038484"/>
+        <origin rpy="0.0 0.0 0.0" xyz="-0.000245 0.000000 -0.007626"/>
+        <inertia ixx="0.000011" ixy="0.000000" ixz="0.000000" iyy="0.000011" iyz="0.000000" izz="0.000021"/>
+      </inertial>
     </link>
     <!-- Following REP199, this frame shall be use to attach EEF or other equipment -->
@@ -115,5 +150,6 @@
       <child link="${prefix}link_1"/>
       <axis xyz="0 0 -1"/>
-      <limit effort="0" lower="${radians(-170)}" upper="${radians(170)}" velocity="${radians(220)}"/>
+      <limit effort="692" lower="${radians(-170)}" upper="${radians(170)}" velocity="${radians(220)}"/>
+      <dynamics damping="0.0" friction="0.0"/>
     </joint>
     <joint name="${prefix}joint_a2" type="revolute">
@@ -122,5 +158,6 @@
       <child link="${prefix}link_2"/>
       <axis xyz="0 1 0"/>
-      <limit effort="0" lower="${radians(-185)}" upper="${radians(65)}" velocity="${radians(210)}"/>
+      <limit effort="574" lower="${radians(-185)}" upper="${radians(65)}" velocity="${radians(210)}"/>
+      <dynamics damping="0.0" friction="0.0"/>
     </joint>
     <joint name="${prefix}joint_a3" type="revolute">
@@ -129,5 +166,6 @@
       <child link="${prefix}link_3"/>
       <axis xyz="0 1 0"/>
-      <limit effort="0" lower="${radians(-137)}" upper="${radians(163)}" velocity="${radians(270)}"/>
+      <limit effort="242" lower="${radians(-137)}" upper="${radians(163)}" velocity="${radians(270)}"/>
+      <dynamics damping="0.0" friction="0.0"/>
     </joint>
     <joint name="${prefix}joint_a4" type="revolute">
@@ -136,5 +174,6 @@
       <child link="${prefix}link_4"/>
       <axis xyz="-1 0 0"/>
-      <limit effort="0" lower="${radians(-185)}" upper="${radians(185)}" velocity="${radians(381)}"/>
+      <limit effort="58" lower="${radians(-185)}" upper="${radians(185)}" velocity="${radians(381)}"/>
+      <dynamics damping="0.0" friction="0.0"/>
     </joint>
     <joint name="${prefix}joint_a5" type="revolute">
@@ -143,5 +182,6 @@
       <child link="${prefix}link_5"/>
       <axis xyz="0 1 0"/>
-      <limit effort="0" lower="${radians(-120)}" upper="${radians(120)}" velocity="${radians(311)}"/>
+      <limit effort="29" lower="${radians(-120)}" upper="${radians(120)}" velocity="${radians(311)}"/>
+      <dynamics damping="0.0" friction="0.0"/>
     </joint>
     <joint name="${prefix}joint_a6" type="revolute">
@@ -150,5 +190,6 @@
       <child link="${prefix}link_6"/>
       <axis xyz="-1 0 0"/>
-      <limit effort="0" lower="${radians(-350)}" upper="${radians(350)}" velocity="${radians(492)}"/>
+      <limit effort="29" lower="${radians(-350)}" upper="${radians(350)}" velocity="${radians(492)}"/>
+      <dynamics damping="0.0" friction="0.0"/>
     </joint>
     <joint name="${prefix}joint_a6-flange" type="fixed">
